Commit message: feat: integrate OpenVINS and detection backends for internal testing
Add classical image detectors, localization selection and observation-only OpenVINS integration. Update desktop configuration and layouts, repair simulation input transport and lifecycle handling, and record registered scene startup checks.

Keep development validation reports local under the updated ignore policy; retain upstream OpenVINS source and patch formatting.

File: src/simulation/easyfly_px4_sitl/models/easyfly_iris/easyfly_iris.urdf (robot description, URDF)
Before this commit: robot easyfly_iris, 5 links, 4 joints
Links:
- added link livox_imu_frame
Joints:
- added joint livox_imu_joint: type fixed, parent livox_frame, child livox_imu_frame, origin xyz=-0.011 -0.02329 -0.00588 rpy=0 0 0
